Commit message: Add IMU link and joint configuration to URDF

File: zyron_description/urdf/zyron.urdf.xacro (robot description, xacro)
@@ -41,4 +41,34 @@
     </collision>
   </link>
+<link name="imu_link">
+  <inertial>
+    <origin xyz="0.0 0.0 0.0" rpy="0.0 0.0 0.0"/>
+    <mass value="0.0"/>
+    <inertia ixx="0.0" ixy="0.0" ixz="0.0" iyy="0.0" iyz="0.0" izz="0.0"/>
+  </inertial>
+  <visual name="">
+    <origin xyz="0.0 0.0 0.0" rpy="0.0 0.0 0.0"/>
+    <geometry>
+      <box size="0.1 0.1 0.1"/>
+    </geometry>
+    <material name="">
+      <color rgba="1.0 0.0 0.0 1.0"/>
+      <texture filename=""/>
+    </material>
+  </visual>
+  <collision>
+    <origin xyz="0.0 0.0 0.0" rpy="0.0 0.0 0.0"/>
+    <geometry>
+      <box size="0.1 0.1 0.1"/>
+    </geometry>
+  </collision>
+</link>
+<joint name="imu_joint" type="fixed">
+  <origin xyz="0.0 0.0 0.0" rpy="0.0 0.0 0.0"/>
+  <parent link="base_link"/>
+  <child link="imu_link"/>
+  <axis xyz="0.0 0.0 0.0"/>
+  <limit lower="0.0" upper="0.0" effort="0.0" velocity="0.0"/>
+</joint>
   <!-- ─── Wheel macro ─────────────────────────────────────────── -->
   <xacro:macro name="wheel" params="name y_offset">
