Commit message: Update robot dimensions and remove unused wheel macro

File: zyron_description/urdf/zyron.urdf.xacro (robot description, xacro)
@@ -5,11 +5,18 @@
   <xacro:arg name="mcu_serial_port" default="/dev/ttyUSB0"/>
   <!-- Robot dimensions (update to match your hardware) -->
-  <xacro:property name="base_length"     value="0.30"/>
-  <xacro:property name="base_width"      value="0.20"/>
-  <xacro:property name="base_height"     value="0.10"/>
+  <xacro:property name="base_length"     value="0.290"/>
+  <xacro:property name="base_width"      value="0.210"/>
+  <xacro:property name="base_height"     value="0.080"/>
   <xacro:property name="wheel_radius"    value="0.033"/>
   <xacro:property name="wheel_width"     value="0.025"/>
-  <xacro:property name="wheel_sep"       value="0.17"/>   <!-- centre-to-centre -->
+  <xacro:property name="wheel_sep"       value="0.245"/>  <!-- centre-to-centre: inner wheel face is 5mm outside body wall -->
   <xacro:property name="caster_radius"   value="0.015"/>
+  <xacro:property name="wheel_x_from_back" value="0.06"/>  <!-- wheels are 6cm from the back edge -->
+  <!-- wheel x in base_link frame: back edge + offset -->
+  <xacro:property name="wheel_x" value="${-base_length/2 + wheel_x_from_back}"/>
+  <!-- Tower on top of base at the back (drive-wheel side), for lidar mount -->
+  <xacro:property name="tower_length"    value="0.120"/>
+  <xacro:property name="tower_width"     value="0.200"/>
+  <xacro:property name="tower_height"    value="0.055"/>
   <!-- ─── base_footprint ─────────────────────────────────────── -->
   <link name="base_footprint"/>
@@ -24,5 +31,5 @@
       <origin xyz="0 0 0" rpy="0 0 0"/>
       <mass value="1.0"/>
-      <inertia ixx="0.0083" ixy="0" ixz="0" iyy="0.0208" iyz="0" izz="0.0250"/>
+      <inertia ixx="0.00421" ixy="0" ixz="0" iyy="0.00754" iyz="0" izz="0.01068"/>
     </inertial>
     <visual>
@@ -31,6 +38,6 @@
         <box size="${base_length} ${base_width} ${base_height}"/>
       </geometry>
-      <material name="blue">
-        <color rgba="0.1 0.2 0.8 1.0"/>
+      <material name="light_grey">
+        <color rgba="0.7 0.7 0.7 1.0"/>
       </material>
     </visual>
@@ -42,4 +49,74 @@
     </collision>
   </link>
+  <!-- ─── Tower (lidar mount platform, back of robot) ────────── -->
+  <link name="tower_link">
+    <inertial>
+      <origin xyz="0 0 0" rpy="0 0 0"/>
+      <mass value="0.2"/>
+      <!-- Solid box inertia: I = m/12*(a²+b²) -->
+      <inertia ixx="0.000327" ixy="0" ixz="0"
+               iyy="0.000733" iyz="0"
+               izz="0.000983"/>
+    </inertial>
+    <visual>
+      <origin xyz="0 0 0" rpy="0 0 0"/>
+      <geometry>
+        <box size="${tower_length} ${tower_width} ${tower_height}"/>
+      </geometry>
+      <material name="light_grey">
+        <color rgba="0.7 0.7 0.7 1.0"/>
+      </material>
+    </visual>
+    <collision>
+      <origin xyz="0 0 0" rpy="0 0 0"/>
+      <geometry>
+        <box size="${tower_length} ${tower_width} ${tower_height}"/>
+      </geometry>
+    </collision>
+  </link>
+  <!-- Tower sits on top of the base, flush with the back (-x) edge -->
+  <!-- x: back edge of base + half tower length = -base_length/2 + tower_length/2 -->
+  <!-- z: top of base + half tower height        =  base_height/2 + tower_height/2 -->
+  <joint name="tower_joint" type="fixed">
+    <parent link="base_link"/>
+    <child  link="tower_link"/>
+    <origin xyz="${-base_length/2 + tower_length/2} 0 ${base_height/2 + tower_height/2}" rpy="0 0 0"/>
+  </joint>
+  <!-- ─── Lidar (mounted on top of tower, centred) ────────────── -->
+  <!-- Dimensions: RPLidar A1 approximate — adjust to your model   -->
+  <xacro:property name="lidar_radius"  value="0.038"/>  <!-- 76mm diameter -->
+  <xacro:property name="lidar_height"  value="0.041"/>  <!-- 41mm tall     -->
+  <link name="lidar_link">
+    <inertial>
+      <origin xyz="0 0 0" rpy="0 0 0"/>
+      <mass value="0.17"/>
+      <!-- Solid cylinder: Ixx=Iyy=m/12*(3r²+h²), Izz=m/2*r² -->
+      <inertia ixx="0.000086" ixy="0" ixz="0"
+               iyy="0.000086" iyz="0"
+               izz="0.000123"/>
+    </inertial>
+    <visual>
+      <origin xyz="0 0 0" rpy="0 0 0"/>
+      <geometry>
+        <cylinder radius="${lidar_radius}" length="${lidar_height}"/>
+      </geometry>
+      <material name="black">
+        <color rgba="0.1 0.1 0.1 1.0"/>
+      </material>
+    </visual>
+    <collision>
+      <origin xyz="0 0 0" rpy="0 0 0"/>
+      <geometry>
+        <cylinder radius="${lidar_radius}" length="${lidar_height}"/>
+      </geometry>
+    </collision>
+  </link>
+  <!-- Lidar sits centred on top of the tower                         -->
+  <!-- z = tower_height/2 (top of tower) + lidar_height/2 (centre)   -->
+  <joint name="lidar_joint" type="fixed">
+    <parent link="tower_link"/>
+    <child  link="lidar_link"/>
+    <origin xyz="0 0 ${tower_height/2 + lidar_height/2}" rpy="0 0 0"/>
+  </joint>
 <link name="imu_link">
   <inertial>
@@ -51,5 +128,5 @@
     <origin xyz="0.0 0.0 0.0" rpy="0.0 0.0 0.0"/>
     <geometry>
-      <box size="0.1 0.1 0.1"/>
+      <box size="0.01 0.01 0.01"/>
     </geometry>
     <material name="">
@@ -61,5 +138,5 @@
     <origin xyz="0.0 0.0 0.0" rpy="0.0 0.0 0.0"/>
     <geometry>
-      <box size="0.1 0.1 0.1"/>
+      <box size="0.01 0.01 0.01"/>
     </geometry>
   </collision>
@@ -99,5 +176,5 @@
       <parent link="base_link"/>
       <child  link="${name}"/>
-      <origin xyz="0 ${y_offset} ${-base_height/2}" rpy="0 0 0"/>
+      <origin xyz="${wheel_x} ${y_offset} ${-base_height/2}" rpy="0 0 0"/>
       <axis xyz="0 1 0"/>
     </joint>
